File: kicad/ATXMEGA256_Miniboard/ATXMEGA256_Miniboard.kicad_sch (KiCad schematic)
At the start: 8 parts, among them U1 ATXMEGA256A3B-AU

Commit message: test
Parts:
- added J1, J2, J3, J4, J5, J6: Conn_01x08_Socket, symbol Connector:Conn_01x08_Socket
- added SW1: SW_Push_Dual, symbol Switch:SW_Push_Dual
Connections:
- net +3V3: no longer C1.2, C2.2, C3.2, C4.2, C5.2, C6.2, U1.15 (VCC_2), U1.25 (VCC_3), U1.35 (VCC_4), U1.45 (VCC_5), U1.53 (VCC), U1.61 (AVCC)
- net at U1.1 (PA3): now also J6.4 (Pin_4)
- net at U1.10 (PB4): now also J5.5 (Pin_5)
- net at U1.11 (PB5): now also J5.6 (Pin_6)
- net at U1.12 (PB6): now also J5.7 (Pin_7)
- net at U1.13 (PB7): now also J5.8 (Pin_8)
- net at U1.16 (PC0): now also J4.1 (Pin_1)
- net at U1.17 (PC1): now also J4.2 (Pin_2)
- net at U1.18 (PC2): now also J4.3 (Pin_3)
- net at U1.19 (PC3): now also J4.4 (Pin_4)
- net at U1.2 (PA4): now also J6.5 (Pin_5)
- net at U1.20 (PC4): now also J4.5 (Pin_5)
- net at U1.21 (PC5): now also J4.6 (Pin_6)
- net at U1.22 (PC6): now also J4.7 (Pin_7)
- net at U1.23 (PC7): now also J4.8 (Pin_8)
- net at U1.26 (PD0): now also J3.1 (Pin_1)
- net at U1.27 (PD1): now also J3.2 (Pin_2)
- net at U1.28 (PD2): now also J3.3 (Pin_3)
- net at U1.29 (PD3): now also J3.4 (Pin_4)
- net at U1.3 (PA5): now also J6.6 (Pin_6)
- net at U1.30 (PD4): now also J3.5 (Pin_5)
- net at U1.31 (PD5): now also J3.6 (Pin_6)
- net at U1.32 (PD6): now also J3.7 (Pin_7)
- net at U1.33 (PD7): now also J3.8 (Pin_8)
- net at U1.36 (PE0): now also J1.1 (Pin_1)
- net at U1.37 (PE1): now also J1.2 (Pin_2)
- net at U1.38 (PE2): now also J1.3 (Pin_3)
- net at U1.39 (PE3): now also J1.4 (Pin_4)
- net at U1.4 (PA6): now also J6.7 (Pin_7)
- net at U1.40 (PE4): now also J1.5 (Pin_5)
- net at U1.41 (PE5): now also J1.6 (Pin_6)
- net at U1.42 (PE6): now also J1.7 (Pin_7)
- net at U1.43 (PE7): now also J1.8 (Pin_8)
- net at U1.46 (PF0): now also J2.1 (Pin_1)
- net at U1.47 (PF1): now also J2.2 (Pin_2)
- net at U1.48 (PF2): now also J2.3 (Pin_3)
- net at U1.49 (PF3): now also J2.4 (Pin_4)
- net at U1.5 (PA7): now also J6.8 (Pin_8)
- net at U1.50 (PF4): now also J2.5 (Pin_5)
- net at U1.51 (PF5): now also J2.6 (Pin_6)
- net at U1.54 (PF6): now also J2.7 (Pin_7)
- net at U1.55 (PF7): now also J2.8 (Pin_8)
- net at U1.6 (PB0): now also J5.1 (Pin_1)
- net at U1.62 (PA0): now also J6.1 (Pin_1)
- net at U1.63 (PA1): now also J6.2 (Pin_2)
- net at U1.64 (PA2): now also J6.3 (Pin_3)
- net at U1.7 (PB1): now also J5.2 (Pin_2)
- net at U1.8 (PB2): now also J5.3 (Pin_3)
- net at U1.9 (PB3): now also J5.4 (Pin_4)
- new net: C4.2, U1.35 (VCC_4)
- new net: C3.2, U1.45 (VCC_5)
- new net: C1.2, U1.53 (VCC)
- new net: C2.2, U1.61 (AVCC)
- new net: C6.2, U1.15 (VCC_2)
- new net: C5.2, U1.25 (VCC_3)

Commit message: magistrale
Parts:
- removed J1, J2, J3, J4, J5, J6: Conn_01x08_Socket, symbol Connector:Conn_01x08_Socket
- added C7, C8: 10p, symbol Device:C
- added J11: Conn_02x05_Counter_Clockwise, symbol Connector_Generic:Conn_02x05_Counter_Clockwise
- added J2: Conn_02x03_Odd_Even, symbol Connector_Generic:Conn_02x03_Odd_Even
- added J7, J8: Conn_01x02_Pin, symbol Connector:Conn_01x02_Pin
- added JP1, JP2: SolderJumper_3_Bridged12, symbol Jumper:SolderJumper_3_Bridged12
- added L1: 2u, symbol Device:L_Ferrite
- added Y1: Crystal_GND2, symbol Device:Crystal_GND2
- added Y2: Crystal_GND24, symbol Device:Crystal_GND24
- C1, C2, C3, C4, C5, C6: value C -> 100n
Connections:
- net +3V3: now also R1.2, J2.2 (Pin_2), J8.2 (Pin_2)
- net GND: now also SW1.1, SW1.3, C7.1, C8.1, J2.6 (Pin_6), Y1.2, Y2.2, Y2.4
- net at C4.2, U1.35 (VCC_4): now also C1.2, C2.2, C3.2, C5.2, U1.15 (VCC_2), U1.25 (VCC_3), U1.45 (VCC_5), U1.53 (VCC), J8.1 (Pin_1), L1.2
- net ~{RESET}: now reaches R1.1
- net ~{RESET}: now also SW1.2, SW1.4, U1.57 (RESET/PDI), J2.5 (Pin_5)
- net PD0: now reaches U1.26 (PD0)
- net PD1: now reaches U1.27 (PD1)
- net PD2: now reaches U1.28 (PD2)
- net PD3: now reaches U1.29 (PD3)
- net PD4: now reaches U1.30 (PD4)
- net PD5: now reaches U1.31 (PD5)
- net PD6: now reaches U1.32 (PD6)
- net PD7: now reaches U1.33 (PD7)
- net PE0: now reaches U1.36 (PE0)
- net PE1: now reaches U1.37 (PE1)
- net PE2: now reaches U1.38 (PE2)
- net PE3: now reaches U1.39 (PE3)
- net PE4: now reaches U1.40 (PE4)
- net PE5: now reaches U1.41 (PE5)
- net at U1.42 (TOSC2): now also Y1.1
- net at U1.43 (TOSC1): now also Y1.3
- net PC0: now reaches U1.16 (PC0)
- net PC1: now reaches U1.17 (PC1)
- net PC2: now reaches U1.18 (PC2)
- net PC3: now reaches U1.19 (PC3)
- net PC4: now reaches U1.20 (PC4)
- net PC5: now reaches U1.21 (PC5)
- net PC6: now reaches U1.22 (PC6)
- net PC7: now reaches U1.23 (PC7)
- net PB0: now reaches U1.6 (PB0)
- net PB1: now reaches U1.7 (PB1)
- net PB2: now reaches U1.8 (PB2)
- net PB3: now reaches U1.9 (PB3)
- net PB4: now reaches U1.10 (PB4)
- net PB5: now reaches U1.11 (PB5)
- net PB6: now reaches U1.12 (PB6)
- net PB7: now reaches U1.13 (PB7)
- net at U1.61 (AVCC): now also C6.2, L1.1; no longer C2.2
- net PF0: now reaches U1.46 (PF0)
- net PF1: now reaches U1.47 (PF1)
- net PF2: now reaches U1.48 (PF2)
- net PF3: now reaches U1.49 (PF3)
- net PF4: now reaches U1.50 (PF4)
- net at U1.51 (VBAT): now also J7.1 (Pin_1)
- net PF6: now reaches U1.54 (PF6)
- net PF7: now reaches U1.55 (PF7)
- net PA3: now reaches U1.1 (PA3)
- net PA4: now reaches U1.2 (PA4)
- net PA5: now reaches U1.3 (PA5)
- net PA6: now reaches U1.4 (PA6)
- net PA7: now reaches U1.5 (PA7)
- net PDI_DATA: now reaches U1.56 (PDI)
- net PDI_DATA: now also J2.1 (Pin_1)
- net PA0: now reaches U1.62 (PA0)
- net PA1: now reaches U1.63 (PA1)
- net PA2: now reaches U1.64 (PA2)
- new net: C7.2, JP1.1 (A), Y2.3
- new net: C8.2, JP2.1 (A), Y2.1
- new net VBAT: J7.2 (Pin_2)
- no-connect marks 0 -> 2
Other:
- moved on the sheet: C1, C2, C3, C4, C5, R1, SW1, U1

Commit message: pierwsza wersja bez nazw i footprintów
Parts:
- removed J11: Conn_02x05_Counter_Clockwise, symbol Connector_Generic:Conn_02x05_Counter_Clockwise
- removed J7, J8: Conn_01x02_Pin, symbol Connector:Conn_01x02_Pin
- added J1, J3, J4, J6, J7: Conn_02x05_Odd_Even, symbol Connector_Generic:Conn_02x05_Odd_Even
- added J5, J8: Conn_02x03_Odd_Even, symbol Connector_Generic:Conn_02x03_Odd_Even
- added JP3, JP4: Jumper_2_Bridged, symbol Jumper:Jumper_2_Bridged
- JP1, JP2: value SolderJumper_3_Bridged12 -> SolderJumper
Connections:
- net +3V3: now also J1.1 (Pin_1), J3.1 (Pin_1), J4.1 (Pin_1), J6.1 (Pin_1), J7.1 (Pin_1), J8.2 (Pin_2), J8.4 (Pin_4), JP4.1 (A)
- net GND: now also J1.10 (Pin_10), J3.10 (Pin_10), J4.10 (Pin_10), J6.10 (Pin_10), J7.10 (Pin_10), J8.3 (Pin_3), J8.5 (Pin_5)
- net PA0: now also J7.3 (Pin_3)
- net PA1: now also J7.2 (Pin_2)
- net PA2: now also J7.5 (Pin_5)
- net PA3: now also J7.4 (Pin_4)
- net PA4: now also J7.7 (Pin_7)
- net PA5: now also J7.6 (Pin_6)
- net PA6: now also J7.9 (Pin_9)
- net PA7: now also J7.8 (Pin_8)
- net PB0: now also J6.3 (Pin_3)
- net PB1: now also J6.2 (Pin_2)
- net PB2: now also J6.5 (Pin_5)
- net PB3: now also J6.4 (Pin_4)
- net PB4: now also J6.7 (Pin_7)
- net PB5: now also J6.6 (Pin_6)
- net PB6: now also J6.9 (Pin_9)
- net PB7: now also J6.8 (Pin_8)
- net PC0: now also J3.3 (Pin_3)
- net PC1: now also J3.2 (Pin_2)
- net PC2: now also J3.5 (Pin_5)
- net PC3: now also J3.4 (Pin_4)
- net PC4: now also J3.7 (Pin_7)
- net PC5: now also J3.6 (Pin_6)
- net PC6: now also J3.9 (Pin_9)
- net PC7: now also J3.8 (Pin_8)
- net PD0: now also J4.3 (Pin_3)
- net PD1: now also J4.2 (Pin_2)
- net PD2: now also J4.5 (Pin_5)
- net PD3: now also J4.4 (Pin_4)
- net PD4: now also J4.7 (Pin_7)
- net PD5: now also J4.6 (Pin_6)
- net PD6: now also J4.9 (Pin_9)
- net PD7: now also J4.8 (Pin_8)
- net PE0: now also J5.1 (Pin_1)
- net PE1: now also J5.2 (Pin_2)
- net PE2: now also J5.3 (Pin_3)
- net PE3: now also J5.4 (Pin_4)
- net PE4: now also J5.5 (Pin_5)
- net PE5: now also J5.6 (Pin_6)
- net PF0: now also J1.3 (Pin_3)
- net PF1: now also J1.2 (Pin_2)
- net PF2: now also J1.5 (Pin_5)
- net PF3: now also J1.4 (Pin_4)
- net PF4: now also J1.7 (Pin_7)
- net PF6: now also J1.9 (Pin_9)
- net PF7: now also J1.8 (Pin_8)
- net VBAT: now also J1.6 (Pin_6), JP3.1 (A)
- net at C1.2, C2.2, C3.2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: now also JP4.2 (B)
- net at JP1.2 (C): now also U1.58 (PR0)
- net at JP1.3 (B): now also J8.1 (Pin_1)
- net at U1.51 (VBAT): now also JP3.2 (B)
- net at JP2.2 (C): now also U1.59 (PR1)
- net at JP2.3 (B): now also J8.6 (Pin_6)
Other:
- moved on the sheet: C1, C2, C3, C4, C5, C6, C7, C8, J2, JP1, JP2, L1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

Commit message: gotowe połączenia oprócz JTAG i kwarców
Parts:
- removed J1, J3: Conn_02x05_Odd_Even, symbol Connector_Generic:Conn_02x05_Odd_Even
- removed SW1: SW_Push_Dual, symbol Switch:SW_Push_Dual
- added J2, J7: ZL264-10DG, Connector_PinSocket_2.54mm:PinSocket_2x05_P2.54mm_Vertical_SMD, symbol Connector_Generic:Conn_02x05_Odd_Even
- added J9: JTAG, Connector_IDC:IDC-Header_2x05_P2.54mm_Vertical, symbol Connector_Generic:Conn_02x05_Odd_Even
- added R2: 330R, Resistor_SMD:R_0805_2012Metric_Pad1.20x1.40mm_HandSolder, symbol Device:R
- added SW1: 1301.9303, symbol Switch:SW_MEC_5E
- C1: renamed from C5; footprint (none) -> Capacitor_SMD:C_0805_2012Metric_Pad1.18x1.45mm_HandSolder
- C2: renamed from C4; footprint (none) -> Capacitor_SMD:C_0805_2012Metric_Pad1.18x1.45mm_HandSolder
- C3, C6: footprint (none) -> Capacitor_SMD:C_0805_2012Metric_Pad1.18x1.45mm_HandSolder
- C4: renamed from C1; footprint (none) -> Capacitor_SMD:C_0805_2012Metric_Pad1.18x1.45mm_HandSolder
- C5: renamed from C2; footprint (none) -> Capacitor_SMD:C_0805_2012Metric_Pad1.18x1.45mm_HandSolder
- C7, C8: footprint (none) -> Capacitor_SMD:C_0603_1608Metric_Pad1.08x0.95mm_HandSolder; Package (none) -> C_0603
- J1: renamed from J2; value Conn_02x03_Odd_Even -> DS1021-2*3SF11-B; footprint (none) -> Connector_PinHeader_2.54mm:PinHeader_2x03_P2.54mm_Vertical_SMD; Manufacturer (none) -> CONNFLY
- J3: renamed from J7; value Conn_02x05_Odd_Even -> ZL264-10DG; footprint (none) -> Connector_PinSocket_2.54mm:PinSocket_2x05_P2.54mm_Vertical_SMD; Manufacturer (none) -> NINIGI
- J4, J6: value Conn_02x05_Odd_Even -> ZL264-10DG; footprint (none) -> Connector_PinSocket_2.54mm:PinSocket_2x05_P2.54mm_Vertical_SMD; Manufacturer (none) -> NINIGI
- J5, J8: value Conn_02x03_Odd_Even -> ZL264-6DG; footprint (none) -> Connector_PinSocket_2.54mm:PinSocket_2x03_P2.54mm_Vertical_SMD; Manufacturer (none) -> NINIGI
- JP1: renamed from JP4; value Jumper_2_Bridged -> DS1021-1X2SF162-B; footprint (none) -> Connector_PinHeader_2.54mm:PinHeader_1x02_P2.54mm_Vertical; Manufacturer (none) -> CONNFLY
- JP2: renamed from JP1; value SolderJumper -> Solder Jumper; footprint (none) -> Jumper:SolderJumper-3_P1.3mm_Bridged12_Pad1.0x1.5mm_NumberLabels; now left out of the parts list
- JP3: value Jumper_2_Bridged -> DS1021-1X2SF162-B; footprint (none) -> Connector_PinHeader_2.54mm:PinHeader_1x02_P2.54mm_Vertical; Manufacturer (none) -> CONNFLY
- JP4: renamed from JP2; value SolderJumper -> Solder Jumper; footprint (none) -> Jumper:SolderJumper-3_P1.3mm_Bridged12_Pad1.0x1.5mm_NumberLabels; now left out of the parts list
- L1: footprint (none) -> Inductor_SMD:L_0805_2012Metric_Pad1.15x1.40mm_HandSolder
- R1: footprint (none) -> Resistor_SMD:R_0805_2012Metric_Pad1.20x1.40mm_HandSolder
- U1: Manufacturer (none) -> Microchip Technology
Connections:
- net +3V3: no longer J1.2 (Pin_2), J3.1 (Pin_1), J4.1 (Pin_1), J6.1 (Pin_1), J8.2 (Pin_2), J8.4 (Pin_4), R1.2
- net GND: now also J4.9 (Pin_9), J2.9 (Pin_9), J7.9 (Pin_9), SW1.1, SW1.2; no longer J4.10 (Pin_10)
- net PC0: now also J2.4 (Pin_4)
- net PC1: now also J2.1 (Pin_1)
- net PC2: now also J2.6 (Pin_6)
- net PC3: now also J2.3 (Pin_3)
- net PC4: now also J2.8 (Pin_8)
- net PC5: now also J2.5 (Pin_5)
- net PC6: now also J2.10 (Pin_10)
- net PC7: now also J2.7 (Pin_7)
- net PD0: now also J4.4 (Pin_4); no longer J4.3 (Pin_3)
- net PD1: now also J4.1 (Pin_1); no longer J4.2 (Pin_2)
- net PD2: now also J4.6 (Pin_6); no longer J4.5 (Pin_5)
- net PD3: now also J4.3 (Pin_3); no longer J4.4 (Pin_4)
- net PD4: now also J4.8 (Pin_8); no longer J4.7 (Pin_7)
- net PD5: now also J4.5 (Pin_5); no longer J4.6 (Pin_6)
- net PD6: now also J4.10 (Pin_10); no longer J4.9 (Pin_9)
- net PD7: now also J4.7 (Pin_7); no longer J4.8 (Pin_8)
- net PF0: now also J7.4 (Pin_4)
- net PF1: now also J7.1 (Pin_1)
- net PF2: now also J7.6 (Pin_6)
- net PF3: now also J7.3 (Pin_3)
- net PF4: now also J7.8 (Pin_8)
- net PF6: now also J7.10 (Pin_10)
- net PF7: now also J7.7 (Pin_7)
- net VBAT: now also J7.5 (Pin_5)
- net ~{RESET}: now also R1.2, R2.2; no longer R1.1
- net at C1.2, C2.2, C3.2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: now also J1.2 (Pin_2), J3.1 (Pin_1), J4.2 (Pin_2), J6.1 (Pin_1), J8.2 (Pin_2), J8.4 (Pin_4), R1.1, J2.2 (Pin_2), J7.2 (Pin_2)
- new net: R2.1, SW1.3 (K), SW1.4 (A)
Other:
- note added: "GPIO Bank A"
- note added: "GPIO Bank B"
- note added: "GPIO Bank C"
- note added: "GPIO Bank D"
- note added: "GPIO Bank E"
- note added: "GPIO Bank F"
- note added: "GPIO Bank R"
- note added: "Kryształ CPU 16MHz"
- note added: "Kryształ RTC 32.768 kHz"
- note added: "Punkt pomiaru prądu VBAT"
- note added: "Punkt pomiaru prądu VCC"
- note added: "Wybór połączenia PR0 - PR1: XTAL/GPIO"
- note added: "Złącze programujące PDI"
- moved on the sheet: C1, C2, C3, C4, C5, C8, J1, J3, J8, JP1, JP2, JP3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

Commit message: v1.0
Parts:
- removed SW1: 1301.9303, symbol Switch:SW_MEC_5E
- added C6: 10u, Capacitor_SMD:C_1210_3225Metric_Pad1.33x2.70mm_HandSolder, symbol Device:C
- added SW1: 1301.9303, Button_Switch_THT:SW_PUSH_6mm_H7.3mm, symbol Switch:SW_Push
- C8: renamed from C7; value 10p -> 12p
- C9: renamed from C8; value 10p -> 12p
- J1: renamed from J9; value JTAG -> DS1013-10SSIB1-B-0; Manufacturer NINIGI -> CONNFLY
- U1: footprint ATXMEGA256A3B-AU:QFP80P1600X1600X120-64N -> ATXMega256A3B-AU:QFP80P1600X1600X120-64N
- Y1: value Crystal_GND2 -> LFXTAL014219; footprint (none) -> Crystal:Crystal_DS26_D2.0mm_L6.0mm_Horizontal_1EP_style1; Manufacturer (none) -> IQD FREQUENCY PRODUCTS
- Y2: value Crystal_GND24 -> LFXTAL053426; footprint (none) -> Crystal:Crystal_SMD_3225-4Pin_3.2x2.5mm; Manufacturer (none) -> IQD FREQUENCY PRODUCTS
- renumbered C6 to C7, J1 to J2, J2 to J3, J3 to J4, J4 to J5, J5 to J6, J6 to J7, J7 to J8, J8 to J9
Connections:
- net GND: now also J1.1 (Pin_1), J1.9 (Pin_9), Y1.3, C6.1, SW1.1; no longer Y1.2
- net PB4: now also J1.6 (Pin_6)
- net PB5: now also J1.10 (Pin_10)
- net PB6: now also J1.2 (Pin_2)
- net PB7: now also J1.4 (Pin_4)
- net ~{RESET}: now also J1.5 (Pin_5)
- net at C1.2, C2.2, C3.2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: now also J1.3 (Pin_3)
- net at R2.1: now also SW1.2
- net at U1.43 (TOSC1): now also Y1.2; no longer Y1.3
- net at C7.2, L1.1, U1.61 (AVCC): now also C6.2
- no-connect marks 2 -> 4
Other:
- note added: "Złącze programujące JTAG"
- moved on the sheet: C1, C2, C3, C4, C5, C7, C8, C9, J1, J2, J3, J4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
