File: kicad/ATXMEGA256_Miniboard/ATXMEGA256_Miniboard.kicad_sch (KiCad schematic)
At the start: 29 parts, among them J1 DS1013-10SSIB1-B-0, J2 DS1021-2*3SF11-B, J3 ZL264-10DG, J4 ZL264-10DG, J5 ZL264-10DG, J6 ZL264-6DG, J7 ZL264-10DG, J8 ZL264-10DG, J9 ZL264-6DG, SW1 1301.9303, U1 ATXMEGA256A3B-AU, Y1 LFXTAL014219, Y2 LFXTAL053426

Commit message: usb + udokumentowanie elementów
Parts:
- removed J3, J5, J7: ZL264-10DG, Connector_PinSocket_2.54mm:PinSocket_2x05_P2.54mm_Vertical_SMD, symbol Connector_Generic:Conn_02x05_Odd_Even
- removed JP1, JP3: DS1021-1X2SF162-B, Connector_PinHeader_2.54mm:PinHeader_1x02_P2.54mm_Vertical, symbol Jumper:Jumper_2_Bridged
- added C10: 4n7, Capacitor_SMD:C_0603_1608Metric_Pad1.08x0.95mm_HandSolder, symbol Device:C
- added J1: 1x3 Goldpin Header, Connector_PinHeader_2.54mm:PinHeader_1x03_P2.54mm_Vertical, symbol Connector:Conn_01x03_Pin
- added J10, J12, J9: 1x2 Goldpin Header, Connector_PinHeader_2.54mm:PinHeader_1x02_P2.54mm_Vertical, symbol Connector:Conn_01x02_Pin
- added J11, J4, J6: 2x5 Goldpin Socket, Connector_PinSocket_2.54mm:PinSocket_2x05_P2.54mm_Vertical_SMD, symbol Connector_Generic:Conn_02x05_Odd_Even
- added J13: USB micro B 2.0 Socket, Connector_USB:USB_Micro-B_Amphenol_10118193-0001LF_Horizontal, symbol Connector:USB_B_Micro
- added R3: 1M, Resistor_SMD:R_0603_1608Metric_Pad0.98x0.95mm_HandSolder, symbol Device:R
- C1, C2, C3, C4, C5, C7: Manufacturer (none) -> KEMET; Package (none) -> C_0805; Part Number (none) -> C0805C104J4RACTU
- C6: Manufacturer (none) -> KEMET; Part Number (none) -> C1210C106K4RAC
- C8: Manufacturer (none) -> KEMET; Part Number (none) -> C0603C120J5GAC
- J14: renamed from J9; value ZL264-6DG -> 2x5 Goldpin Socket; Part Number (none) -> ZL264-6DG
- J2: renamed from J1; value DS1013-10SSIB1-B-0 -> 2x5 IDC Socket; Part Number (none) -> DS1013-10SSIB1-B-0
- J3: renamed from J2; value DS1021-2*3SF11-B -> 2x5 Goldpin Header; Part Number (none) -> DS1021-2*3SF11-B
- J5: renamed from J4; value ZL264-10DG -> 2x5 Goldpin Socket; Part Number (none) -> ZL264-10DG
- J7: renamed from J6; value ZL264-6DG -> 2x3 Goldpin Socket; Part Number (none) -> ZL264-6DG
- J8: value ZL264-10DG -> 2x5 Goldpin Socket; Part Number (none) -> ZL264-10DG
- L1: value 2u -> 2u2; Manufacturer (none) -> TDK; Package (none) -> L_0805; Part Number (none) -> MLZ2012A2R2WT000
- R1: footprint Resistor_SMD:R_0805_2012Metric_Pad1.20x1.40mm_HandSolder -> Resistor_SMD:R_0603_1608Metric_Pad0.98x0.95mm_HandSolder; Manufacturer (none) -> ROYAL OHM; Package (none) -> R_0603; Part Number (none) -> 0603SAJ0103T5E
- R2: footprint Resistor_SMD:R_0805_2012Metric_Pad1.20x1.40mm_HandSolder -> Resistor_SMD:R_0603_1608Metric_Pad0.98x0.95mm_HandSolder; Manufacturer (none) -> ROYAL OHM; Package (none) -> R_0603; Part Number (none) -> 0603SAJ0331T5E
- SW1: Part Number (none) -> 1301.9303
- U1: Availability In Stock -> (none); Check_prices https://www.snapeda.com/parts/ATXMEGA256A3B-AU/Microchip/vi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 -> (none); DESCRIPTION 8/16-bit XMEGA A3 Microcontroller -> (none); MF Microchip Technology -> (none); MP ATXMEGA256A3B-AU -> (none); MPN ATXMEGA256A3B-AU -> (none); Manufacturer Microchip Technology -> Microchip; OC_FARNELL 1841632 -> (none); OC_NEWARK - -> (none); PACKAGE TQFP-64 -> (none); Package TQFP-64 Microchip -> TQFP-64; Part Number (none) -> ATXMEGA256A3B-AU; Price None -> (none); SUPPLIER Atmel Corporation -> (none); SnapEDA_Link https://www.snapeda.com/parts/ATXMEGA256A3B-AU/Microchip/vi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 -> (none)
- Y1: value LFXTAL014219 -> 32.768 kHz; Package (none) -> THT_D2.0mm_L6.0mm; Part Number (none) -> LFXTAL014219
- Y2: value LFXTAL053426 -> 16 MHz; Package (none) -> SMD_4Pin_3.2x2.5mm; Part Number (none) -> LFXTAL053426
- renumbered JP2 to JP1, JP4 to JP2
Connections:
- net +3V3: now also J1.3 (Pin_3)
- net GND: now also J8.10 (Pin_10), C10.1, J11.9 (Pin_9), J13.5 (GND), J4.9 (Pin_9), J6.9 (Pin_9), R3.2; no longer J8.9 (Pin_9)
- net PB0: now also J8.3 (Pin_3)
- net PB1: now also J8.2 (Pin_2)
- net PB2: now also J8.5 (Pin_5)
- net PB3: now also J8.4 (Pin_4)
- net PB4: now also J8.7 (Pin_7)
- net PB5: now also J8.6 (Pin_6)
- net PB6: now also J8.9 (Pin_9)
- net PB7: now also J8.8 (Pin_8)
- net PC0: now also J4.4 (Pin_4)
- net PC1: now also J4.1 (Pin_1)
- net PC2: now also J4.6 (Pin_6)
- net PC3: now also J4.3 (Pin_3)
- net PC4: now also J4.8 (Pin_8)
- net PC5: now also J4.5 (Pin_5)
- net PC6: now also J4.10 (Pin_10)
- net PC7: now also J4.7 (Pin_7)
- net PD0: now also J6.4 (Pin_4)
- net PD1: now also J6.1 (Pin_1)
- net PD2: now also J6.6 (Pin_6)
- net PD3: now also J6.3 (Pin_3)
- net PD4: now also J6.8 (Pin_8)
- net PD5: now also J6.5 (Pin_5)
- net PF0: now also J11.4 (Pin_4); no longer J8.4 (Pin_4)
- net PF1: now also J11.1 (Pin_1); no longer J8.1 (Pin_1)
- net PF2: now also J11.6 (Pin_6); no longer J8.6 (Pin_6)
- net PF3: now also J11.3 (Pin_3); no longer J8.3 (Pin_3)
- net PF4: now also J11.8 (Pin_8); no longer J8.8 (Pin_8)
- net PF6: now also J11.10 (Pin_10); no longer J8.10 (Pin_10)
- net PF7: now also J11.7 (Pin_7); no longer J8.7 (Pin_7)
- net VBAT: now also J11.5 (Pin_5), J12.2 (Pin_2); no longer J8.5 (Pin_5)
- net at C1.2, C2.2, C3.2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: now also J8.1 (Pin_1), J1.2 (Pin_2), J11.2 (Pin_2), J4.2 (Pin_2), J6.2 (Pin_2); no longer J8.2 (Pin_2)
- net at U1.51 (VBAT): now also J12.1 (Pin_1)
- net PD6 renamed D-
- net D-: now also J6.10 (Pin_10), J9.1 (Pin_1)
- net PD7 renamed D+
- net D+: now also J10.1 (Pin_1), J6.7 (Pin_7)
- new net: J10.2 (Pin_2), J13.3 (D+)
- new net: J13.2 (D-), J9.2 (Pin_2)
- new net: C10.2, J13.6 (Shield), R3.1
- new net +5V: J13.1 (VBUS)
- new net VCC: J1.1 (Pin_1)
- no-connect marks 4 -> 5
Other:
- note added: "Kryształ CPU"
- note added: "Kryształ RTC"
- note added: "Przycisk RESET"
- note added: "Punkt pomiaru prądu I_BAT"
- note added: "Wybór połączenia PB6- PB7: USB/GPIO"
- note added: "Wybór źródła zasilania: z regulatora / zewnętrzne"
- note added: "Złącze USB"
- note removed: "Kryształ CPU 16MHz"
- note removed: "Kryształ RTC 32.768 kHz"
- note removed: "Punkt pomiaru prądu VBAT"
- note removed: "Punkt pomiaru prądu VCC"
- moved on the sheet: C1, C6, C8, C9, J14, J2, J3, J5, J7, JP1, JP2, L1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

Commit message: poprawka nazwy headera
Parts:
- J14: value 2x5 Goldpin Socket -> 2x3 Goldpin Socket
- J3: value 2x5 Goldpin Header -> 2x3 Goldpin Header
Changed lines of the file:
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@@
       (effects (font (size 1.27 1.27)))
     )
-    (property "Value" "2x5 Goldpin Socket" (at 90.17 172.72 0)
+    (property "Value" "2x3 Goldpin Socket" (at 90.17 172.72 0)
       (effects (font (size 1.27 1.27)))
     )
@@
       (effects (font (size 1.27 1.27)))
     )
-    (property "Value" "2x5 Goldpin Header" (at 247.65 48.26 0)
-      (effects (font (size 1.27 1.27)))
-    )
+    (property "Value" "2x3 Goldpin Header" (at 247.65 48.26 0)
+      (effects (font (size 1.27 1.27)))
+    )

Commit message: przycisk zmieniony na smd
Parts:
- SW1: value 1301.9303 -> Microswitch; footprint Button_Switch_THT:SW_PUSH_6mm_H7.3mm -> Button_Switch_SMD:SW_SPST_Omron_B3FS-100xP; Manufacturer SCHURTER -> KNITTER-SWITCH; Part Number 1301.9303 -> TSS62N
Changed lines of the file:
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@@
     (effects (font (size 1.27 1.27)) (justify left bottom))
   )
-  (label "PD7" (at 269.24 106.68 0)
+  (label "PD7" (at 269.24 106.68 0) (fields_autoplaced)
     (effects (font (size 1.27 1.27)) (justify left bottom))
   )
@@
     (effects (font (size 1.27 1.27)) (justify right bottom))
   )
-  (label "PD6" (at 269.24 109.22 0)
+  (label "PD6" (at 269.24 109.22 0) (fields_autoplaced)
     (effects (font (size 1.27 1.27)) (justify left bottom))
   )
@@
       (effects (font (size 1.27 1.27)))
     )
-    (property "Value" "1301.9303" (at 109.22 71.12 0)
-      (effects (font (size 1.27 1.27)))
-    )
-    (property "Footprint" "Button_Switch_THT:SW_PUSH_6mm_H7.3mm" (at 109.22 71.12 0)
+    (property "Value" "Microswitch" (at 109.22 71.12 0)
+      (effects (font (size 1.27 1.27)))
+    )
+    (property "Footprint" "Button_Switch_SMD:SW_SPST_Omron_B3FS-100xP" (at 109.22 71.12 0)
       (effects (font (size 1.27 1.27)) hide)
     )
@@
       (effects (font (size 1.27 1.27)) hide)
     )
-    (property "Part Number" "1301.9303" (at 109.22 76.2 0)
-      (effects (font (size 1.27 1.27)) hide)
-    )
-    (property "Manufacturer" "SCHURTER" (at 109.22 76.2 0)
-      (effects (font (size 1.27 1.27)) hide)
-    )
+    (property "Part Number" "TSS62N" (at 109.22 76.2 0)
+      (effects (font (size 1.27 1.27)) hide)
+    )
+    (property "Manufacturer" "KNITTER-SWITCH" (at 109.22 76.2 0)
+      (effects (font (size 1.27 1.27)) hide)
+    )

Commit message: zasilanie
Parts:
- removed J1: 1x3 Goldpin Header, Connector_PinHeader_2.54mm:PinHeader_1x03_P2.54mm_Vertical, symbol Connector:Conn_01x03_Pin
- C9: Manufacturer (none) -> KEMET; Part Number (none) -> C0603C120J5GAC
- renumbered J2 to J1, J11 to J10, J12 to J11, J13 to J12, J14 to J13, J3 to J2, J4 to J3, J5 to J4, J6 to J5, J7 to J6, J8 to J7, J9 to J8, J10 to J9
Connections:
- net VCC: now also C1.2, C2.2, C3.2, C4.2, C5.2, J1.3 (Pin_3), J10.2 (Pin_2), J13.2 (Pin_2), J13.4 (Pin_4), J2.2 (Pin_2), J3.2 (Pin_2), J4.1 (Pin_1), J5.2 (Pin_2), J7.1 (Pin_1), L1.2, R1.1, U1.15 (VCC_2), U1.25 (VCC_3), U1.35 (VCC_4), U1.45 (VCC_5), U1.53 (VCC)
Other:
- added sheet Power Supply (power_supply.kicad_sch)
- note added: "Rezonator CPU"
- note added: "Rezonator RTC"
- note removed: "Kryształ CPU"
- note removed: "Kryształ RTC"
- note removed: "Wybór źródła zasilania: z regulatora / zewnętrzne"
- moved on the sheet: J11

Commit message: led + złącze masy + złącze śrubowe (do opisania)
Parts:
- added J14: 2x3 Goldpin Socket, Connector_PinSocket_2.54mm:PinSocket_2x03_P2.54mm_Vertical_SMD, symbol Connector_Generic:Conn_02x03_Odd_Even
- C1, C2, C3, C4, C5, C7: Package C_0805 -> 0805
- C10, C8, C9: Package C_0603 -> 0603
- C6: Package C_1210 -> 1210
- L1: Package L_0805 -> 0805
- R1, R2, R3: Package R_0603 -> 0603
- U1: footprint ATXMega256A3B-AU:QFP80P1600X1600X120-64N -> ATXMEGA256A3B-AU:QFP80P1600X1600X120-64N
Connections:
- net GND: now also J14.1 (Pin_1), J14.2 (Pin_2), J14.3 (Pin_3), J14.4 (Pin_4), J14.5 (Pin_5), J14.6 (Pin_6)
- net VCC renamed +3V3
Other:
- sheet Power Supply ports: added +3V3, +5V; removed none

Commit message: poprawka estetyczna zasilania
Parts:
- added J17: Screw_Terminal_01x02, symbol Connector:Screw_Terminal_01x02
- U1: footprint ATXMEGA256A3B-AU:QFP80P1600X1600X120-64N -> ATXMega256A3B-AU:QFP80P1600X1600X120-64N
Connections:
- net GND: now also J17.1 (Pin_1)
- new net Power Supply/EXT_VCC: J17.2 (Pin_2)
Other:
- sheet Power Supply ports: added EXT_VCC; removed none
- note added: "Zasilanie zewnętrzne 5 - 16 V"
Changed lines of the file:
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@@
+    (stroke (width 0) (type default))
+  )
+  (wire (pts (xy 44.45 34.29) (xy 39.37 34.29))
     (stroke (width 0) (type default))
   )
@@
     (stroke (width 0) (type default))
   )
+  (wire (pts (xy 54.61 31.75) (xy 39.37 31.75))
+    (stroke (width 0) (type default))
+  )
   (wire (pts (xy 142.24 147.32) (xy 140.97 147.32))
     (stroke (width 0) (type default))
@@
     (stroke (width 0) (type default))
   )
-  (wire (pts (xy 52.07 29.21) (xy 62.23 29.21))
+  (wire (pts (xy 74.93 29.21) (xy 85.09 29.21))
     (stroke (width 0) (type default))
   )
@@
     (stroke (width 0) (type default))
   )
-  (wire (pts (xy 62.23 29.21) (xy 62.23 21.59))
+  (wire (pts (xy 85.09 29.21) (xy 85.09 21.59))
     (stroke (width 0) (type default))
   )
@@
     (stroke (width 0) (type default))
   )
-  (wire (pts (xy 31.75 29.21) (xy 22.86 29.21))
+  (wire (pts (xy 54.61 25.4) (xy 45.72 25.4))
     (stroke (width 0) (type default))
   )
@@
     (stroke (width 0) (type default))
   )
+  (wire (pts (xy 44.45 39.37) (xy 44.45 34.29))
+    (stroke (width 0) (type default))
+  )
   (wire (pts (xy 29.21 63.5) (xy 40.64 63.5))
     (stroke (width 0) (type default))
@@
     (stroke (width 0) (type default))
   )
-  (wire (pts (xy 22.86 29.21) (xy 22.86 21.59))
+  (wire (pts (xy 45.72 25.4) (xy 45.72 21.59))
     (stroke (width 0) (type default))
   )
@@
   )
   (text "GPIO Bank D" (at 259.08 96.52 90)
+    (effects (font (size 1.27 1.27)) (justify left bottom))
+  )
+  (text "Zasilanie\nzewnętrzne\n5 - 16 V" (at 19.05 36.83 0)
     (effects (font (size 1.27 1.27)) (justify left bottom))
   )
@@
     )
   )
+  (symbol (lib_id "Connector:Screw_Terminal_01x02") (at 34.29 34.29 180) (unit 1)
+    (in_bom yes) (on_board yes) (dnp no) (fields_autoplaced)
+    (property "Reference" "J17" (at 34.29 25.4 0)
+      (effects (font (size 1.27 1.27)))
+    )
+    (property "Value" "Screw_Terminal_01x02" (at 34.29 27.94 0)
+      (effects (font (size 1.27 1.27)))
+    )
+    (property "Footprint" "" (at 34.29 34.29 0)
+      (effects (font (size 1.27 1.27)) hide)
+    )
+    (property "Datasheet" "~" (at 34.29 34.29 0)
+      (effects (font (size 1.27 1.27)) hide)
+    )
+    (pin "1")
+    (pin "2")
+    (instances
+      (project "ATXMEGA256_Miniboard"
+        (path "/ef1e5883-c6cf-4bad-8eaa-8ec9109f9d71"
+          (reference "J17") (unit 1)
+        )
+      )
+    )
+  )
   (symbol (lib_id "Device:C") (at 63.5 71.12 180) (unit 1)
     (in_bom yes) (on_board yes) (dnp no)
@@
         (path "/ef1e5883-c6cf-4bad-8eaa-8ec9109f9d71"
           (reference "#PWR04") (unit 1)
+        )
+      )
+    )
+  )
+  (symbol (lib_id "power:GND") (at 44.45 39.37 0) (unit 1)
+    (in_bom yes) (on_board yes) (dnp no) (fields_autoplaced)
+    (property "Reference" "#PWR013" (at 44.45 45.72 0)
+      (effects (font (size 1.27 1.27)) hide)
+    )
+    (property "Value" "GND" (at 44.45 44.45 0)
+      (effects (font (size 1.27 1.27)))
+    )
+    (property "Footprint" "" (at 44.45 39.37 0)
+      (effects (font (size 1.27 1.27)) hide)
+    )
+    (property "Datasheet" "" (at 44.45 39.37 0)
+      (effects (font (size 1.27 1.27)) hide)
+    )
+    (pin "1")
+    (instances
+      (project "ATXMEGA256_Miniboard"
+        (path "/ef1e5883-c6cf-4bad-8eaa-8ec9109f9d71"
+          (reference "#PWR013") (unit 1)
         )
       )
@@
     )
   )
-  (symbol (lib_id "power:+5V") (at 22.86 21.59 0) (unit 1)
-    (in_bom yes) (on_board yes) (dnp no) (fields_autoplaced)
-    (property "Reference" "#PWR01" (at 22.86 25.4 0)
-      (effects (font (size 1.27 1.27)) hide)
-    )
-    (property "Value" "+5V" (at 22.86 16.51 0)
-      (effects (font (size 1.27 1.27)))
-    )
-    (property "Footprint" "" (at 22.86 21.59 0)
-      (effects (font (size 1.27 1.27)) hide)
-    )
-    (property "Datasheet" "" (at 22.86 21.59 0)
+  (symbol (lib_id "power:+5V") (at 45.72 21.59 0) (unit 1)
+    (in_bom yes) (on_board yes) (dnp no) (fields_autoplaced)
+    (property "Reference" "#PWR01" (at 45.72 25.4 0)
+      (effects (font (size 1.27 1.27)) hide)
+    )
+    (property "Value" "+5V" (at 45.72 16.51 0)
+      (effects (font (size 1.27 1.27)))
+    )
+    (property "Footprint" "" (at 45.72 21.59 0)
+      (effects (font (size 1.27 1.27)) hide)
+    )
+    (property "Datasheet" "" (at 45.72 21.59 0)
       (effects (font (size 1.27 1.27)) hide)
     )
@@
       (effects (font (size 1.27 1.27)))
     )
-    (property "Footprint" "ATXMEGA256A3B-AU:QFP80P1600X1600X120-64N" (at 162.56 96.52 0)
+    (property "Footprint" "ATXMega256A3B-AU:QFP80P1600X1600X120-64N" (at 162.56 96.52 0)
       (effects (font (size 1.27 1.27)) (justify bottom) hide)
     )
@@
     )
   )
-  (symbol (lib_id "power:+3V3") (at 62.23 21.59 0) (unit 1)
-    (in_bom yes) (on_board yes) (dnp no) (fields_autoplaced)
-    (property "Reference" "#PWR02" (at 62.23 25.4 0)
-      (effects (font (size 1.27 1.27)) hide)
-    )
-    (property "Value" "+3V3" (at 62.23 16.51 0)
-      (effects (font (size 1.27 1.27)))
-    )
-    (property "Footprint" "" (at 62.23 21.59 0)
-      (effects (font (size 1.27 1.27)) hide)
-    )
-    (property "Datasheet" "" (at 62.23 21.59 0)
+  (symbol (lib_id "power:+3V3") (at 85.09 21.59 0) (unit 1)
+    (in_bom yes) (on_board yes) (dnp no) (fields_autoplaced)
+    (property "Reference" "#PWR02" (at 85.09 25.4 0)
+      (effects (font (size 1.27 1.27)) hide)
+    )
+    (property "Value" "+3V3" (at 85.09 16.51 0)
+      (effects (font (size 1.27 1.27)))
+    )
+    (property "Footprint" "" (at 85.09 21.59 0)
+      (effects (font (size 1.27 1.27)) hide)
+    )
+    (property "Datasheet" "" (at 85.09 21.59 0)
       (effects (font (size 1.27 1.27)) hide)
     )
@@
     )
   )
-  (sheet (at 31.75 21.59) (size 20.32 13.97) (fields_autoplaced)
+  (sheet (at 54.61 21.59) (size 20.32 13.97) (fields_autoplaced)
     (stroke (width 0.1524) (type solid))
     (fill (color 0 0 0 0.0000))
-    (property "Sheetname" "Power Supply" (at 31.75 20.8784 0)
+    (property "Sheetname" "Power Supply" (at 54.61 20.8784 0)
       (effects (font (size 1.27 1.27)) (justify left bottom))
     )
-    (property "Sheetfile" "power_supply.kicad_sch" (at 31.75 36.1446 0)
+    (property "Sheetfile" "power_supply.kicad_sch" (at 54.61 36.1446 0)
       (effects (font (size 1.27 1.27)) (justify left top))
     )
-    (pin "+5V" input (at 31.75 29.21 180)
+    (pin "+5V" input (at 54.61 25.4 180)
       (effects (font (size 1.27 1.27)) (justify left))
     )
-    (pin "+3V3" input (at 52.07 29.21 0)
+    (pin "+3V3" input (at 74.93 29.21 0)
       (effects (font (size 1.27 1.27)) (justify right))
     )
-    (instances
+    (pin "EXT_VCC" input (at 54.61 31.75 180)
+      (effects (font (size 1.27 1.27)) (justify left))
+    )
+    (instances

Commit message: schemat rev. 1.0
Parts:
- removed C1, C2, C3, C4, C5, C7: 100n, Capacitor_SMD:C_0805_2012Metric_Pad1.18x1.45mm_HandSolder, symbol Device:C
- removed C6: 10u, Capacitor_SMD:C_1210_3225Metric_Pad1.33x2.70mm_HandSolder, symbol Device:C
- removed L1: 2u2, Inductor_SMD:L_0805_2012Metric_Pad1.15x1.40mm_HandSolder, symbol Device:L_Ferrite
- J2: renamed from J17; value Screw_Terminal_01x02 -> 1x2 Screw Terminal; footprint (none) -> TerminalBlock_4Ucon:TerminalBlock_4Ucon_1x02_P3.50mm_Horizontal; Manufacturer (none) -> DEGSON ELECTRONICS; Part Number (none) -> DG381-3.5-02P-13-00AH
- SW1: value Microswitch -> RESET
- renumbered C8 to C1, C9 to C2, C10 to C3, J9 to J10, J10 to J11, J11 to J12, J12 to J13, J13 to J14, J14 to J15, J2 to J3, J3 to J4, J4 to J5, J5 to J6, J6 to J7, J7 to J8, J8 to J9
Connections:
- net +3V3: no longer R1.1, U1.15 (VCC_2), U1.25 (VCC_3), U1.35 (VCC_4), U1.45 (VCC_5), U1.53 (VCC)
- net Power Supply/+3V3_MCU_AVCC: now reaches U1.61 (AVCC)
- new net Power Supply/+3V3_MCU_VCC: R1.1, U1.15 (VCC_2), U1.25 (VCC_3), U1.35 (VCC_4), U1.45 (VCC_5), U1.53 (VCC)
Other:
- sheet Power Supply ports: added +3V3_MCU_AVCC, +3V3_MCU_VCC; removed none
- note added: "Zasilanie zewnętrzne 4.3 - 16 V"
- note removed: "Przycisk RESET"
- note removed: "Zasilanie zewnętrzne 5 - 16 V"
- moved on the sheet: J2, R1

Commit message: optymalizacja BOM + pdf schematu
Parts:
- removed R2: 330R, Resistor_SMD:R_0603_1608Metric_Pad0.98x0.95mm_HandSolder, symbol Device:R
- J13: Part Number 101181930001LF -> 10118192-0001LF
- J2: footprint TerminalBlock_4Ucon:TerminalBlock_4Ucon_1x02_P3.50mm_Horizontal -> TerminalBlock:TerminalBlock_bornier-2_P5.08mm
- SW1: Manufacturer KNITTER-SWITCH -> TE Connectivity; Part Number TSS62N -> FSM2JSMAA
- renumbered R3 to R2
Connections:
- net ~{RESET}: now also SW1.2
Changed lines of the file:
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@@
-    (stroke (width 0) (type default))
-  )
-  (wire (pts (xy 125.73 76.2) (xy 128.27 76.2))
     (stroke (width 0) (type default))
   )
@@
     (stroke (width 0) (type default))
   )
-  (wire (pts (xy 114.3 76.2) (xy 118.11 76.2))
+  (wire (pts (xy 114.3 76.2) (xy 128.27 76.2))
     (stroke (width 0) (type default))
   )
@@
       (effects (font (size 1.27 1.27)))
     )
-    (property "Footprint" "TerminalBlock_4Ucon:TerminalBlock_4Ucon_1x02_P3.50mm_Horizontal" (at 34.29 49.53 0)
+    (property "Footprint" "TerminalBlock:TerminalBlock_bornier-2_P5.08mm" (at 34.29 49.53 0)
       (effects (font (size 1.27 1.27)) hide)
     )
@@
     )
   )
-  (symbol (lib_id "Device:R") (at 121.92 76.2 90) (unit 1)
-    (in_bom yes) (on_board yes) (dnp no)
-    (property "Reference" "R2" (at 121.92 69.85 90)
-      (effects (font (size 1.27 1.27)))
-    )
-    (property "Value" "330R" (at 121.92 72.39 90)
-      (effects (font (size 1.27 1.27)))
-    )
-    (property "Footprint" "Resistor_SMD:R_0603_1608Metric_Pad0.98x0.95mm_HandSolder" (at 121.92 77.978 90)
-      (effects (font (size 1.27 1.27)) hide)
-    )
-    (property "Datasheet" "~" (at 121.92 76.2 0)
-      (effects (font (size 1.27 1.27)) hide)
-    )
-    (property "Part Number" "0603SAJ0331T5E" (at 121.92 76.2 90)
-      (effects (font (size 1.27 1.27)) hide)
-    )
-    (property "Manufacturer" "ROYAL OHM" (at 121.92 76.2 90)
-      (effects (font (size 1.27 1.27)) hide)
-    )
-    (property "Package" "0603" (at 121.92 78.74 90)
-      (effects (font (size 1.27 1.27)) hide)
-    )
-    (pin "2")
-    (pin "1")
-    (instances
-      (project "ATXMEGA256_Miniboard"
-        (path "/ef1e5883-c6cf-4bad-8eaa-8ec9109f9d71"
-          (reference "R2") (unit 1)
-        )
-      )
-    )
-  )
   (symbol (lib_id "Connector_Generic:Conn_02x03_Odd_Even") (at 246.38 54.61 0) (unit 1)
     (in_bom yes) (on_board yes) (dnp no) (fields_autoplaced)
@@
   (symbol (lib_id "Device:R") (at 35.56 175.26 0) (mirror y) (unit 1)
     (in_bom yes) (on_board yes) (dnp no)
-    (property "Reference" "R3" (at 33.02 173.99 0)
+    (property "Reference" "R2" (at 33.02 173.99 0)
       (effects (font (size 1.27 1.27)) (justify left))
     )
@@
       (project "ATXMEGA256_Miniboard"
         (path "/ef1e5883-c6cf-4bad-8eaa-8ec9109f9d71"
-          (reference "R3") (unit 1)
+          (reference "R2") (unit 1)
         )
       )
@@
       (effects (font (size 1.27 1.27)) hide)
     )
-    (property "Part Number" "101181930001LF" (at 38.1 156.21 0)
+    (property "Part Number" "10118192-0001LF" (at 38.1 156.21 0)
       (effects (font (size 1.27 1.27)) hide)
     )
@@
       (effects (font (size 1.27 1.27)) hide)
     )
-    (property "Part Number" "TSS62N" (at 109.22 76.2 0)
-      (effects (font (size 1.27 1.27)) hide)
-    )
-    (property "Manufacturer" "KNITTER-SWITCH" (at 109.22 76.2 0)
-      (effects (font (size 1.27 1.27)) hide)
-    )
+    (property "Part Number" "FSM2JSMAA" (at 109.22 76.2 0)
+      (effects (font (size 1.27 1.27)) hide)
+    )
+    (property "Manufacturer" "TE Connectivity" (at 109.22 76.2 0)
+      (effects (font (size 1.27 1.27)) hide)
+    )
