File: kicad/ATXMEGA256_Miniboard/ATXMEGA256_Miniboard.kicad_sch (KiCad schematic)
At the start: 25 parts, among them J1 10118192-0001LF, J2 2x5 IDC Socket, J3 2x3 IDC Socket, SW1 RESET, U1 ATXMEGA256A3B-AU, Y1 32.768 kHz, Y2 16 MHz

Commit message: wstepne poczenia
Parts:
- removed SW1: RESET, FSM2JSMAA:SW_SMD_2-1437565-8_4_4.50_6.00_6.00_5.00, symbol Switch:SW_Push
- added SW1: RESET, FSM2JSMAA:SW_SMD_2-1437565-8_4_4.50_6.00_6.00_5.00, symbol Switch:SW_MEC_5E
Connections:
- net GND: now also SW1.1, SW1.2
- net ~{RESET}: now also SW1.3 (K), SW1.4 (A)
- net MCU_AVCC: now reaches C6.2, C7.2, L1.2, U1.61 (AVCC)
Changed lines of the file:
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@@
 	)
 	(junction
+		(at 50.8 86.36)
+		(diameter 0)
+		(color 0 0 0 0)
+	)
+	(junction
 		(at 62.23 34.29)
 		(diameter 0)
@@
 	(wire
 		(pts
-			(xy 106.68 59.69) (xy 93.98 59.69)
-		)
-		(stroke
-			(width 0)
-			(type default)
-		)
-	)
-	(wire
-		(pts
 			(xy 144.78 115.57) (xy 143.51 115.57)
 		)
@@
 	(wire
 		(pts
+			(xy 50.8 86.36) (xy 53.34 86.36)
+		)
+		(stroke
+			(width 0)
+			(type default)
+		)
+	)
+	(wire
+		(pts
 			(xy 135.89 59.69) (xy 144.78 59.69)
 		)
@@
 	(wire
 		(pts
+			(xy 50.8 100.33) (xy 53.34 100.33)
+		)
+		(stroke
+			(width 0)
+			(type default)
+		)
+	)
+	(wire
+		(pts
 			(xy 217.17 113.03) (xy 217.17 114.3)
 		)
@@
 	(wire
 		(pts
-			(xy 45.72 86.36) (xy 53.34 86.36)
+			(xy 43.18 86.36) (xy 50.8 86.36)
 		)
 		(stroke
@@
 	(wire
 		(pts
+			(xy 50.8 86.36) (xy 50.8 88.9)
+		)
+		(stroke
+			(width 0)
+			(type default)
+		)
+	)
+	(wire
+		(pts
 			(xy 135.89 95.25) (xy 144.78 95.25)
 		)
@@
 	(wire
 		(pts
+			(xy 50.8 99.06) (xy 50.8 100.33)
+		)
+		(stroke
+			(width 0)
+			(type default)
+		)
+	)
+	(wire
+		(pts
 			(xy 143.51 39.37) (xy 143.51 36.83)
 		)
@@
 		)
 	)
+	(wire
+		(pts
+			(xy 93.98 59.69) (xy 106.68 59.69)
+		)
+		(stroke
+			(width 0)
+			(type default)
+		)
+	)
 	(bus
 		(pts
@@
 	)
 	(label "~{RESET}"
-		(at 45.72 86.36 0)
+		(at 43.18 86.36 0)
 		(effects
 			(font
@@
 		)
 	)
+	(label "MCU_AVCC"
+		(at 95.25 59.69 0)
+		(effects
+			(font
+				(size 1.27 1.27)
+			)
+			(justify left bottom)
+		)
+	)
 	(label "PC4"
 		(at 190.5 44.45 0)
@@
 	)
 	(symbol
-		(lib_id "Switch:SW_Push")
+		(lib_id "Switch:SW_MEC_5E")
 		(at 53.34 93.98 90)
 		(unit 1)
@@
 		(fields_autoplaced yes)
 		(property "Reference" "SW1"
-			(at 54.61 92.71 90)
+			(at 54.61 92.7099 90)
 			(effects
 				(font
@@
 		)
 		(property "Value" "RESET"
-			(at 54.61 95.25 90)
+			(at 54.61 95.2499 90)
 			(effects
 				(font
@@
 		)
 		(property "Footprint" "FSM2JSMAA:SW_SMD_2-1437565-8_4_4.50_6.00_6.00_5.00"
-			(at 48.26 93.98 0)
+			(at 45.72 93.98 0)
 			(effects
 				(font
@@
 			)
 		)
-		(property "Datasheet" "~"
-			(at 48.26 93.98 0)
+		(property "Datasheet" ""
+			(at 45.72 93.98 0)
 			(effects
 				(font
@@
 					(size 1.27 1.27)
 				)
+				(hide yes)
 			)
 		)
@@
 			)
 		)
+		(pin "2"
+		)
+		(pin "3"
+		)
 		(pin "1"
 		)
-		(pin "2"
+		(pin "4"
 		)
 		(instances
-			(project "ATXMEGA256_Miniboard"
+			(project ""
 				(path "/ef1e5883-c6cf-4bad-8eaa-8ec9109f9d71"
 					(reference "SW1")
