File: kicad/ATXMEGA256_Miniboard/power_supply.kicad_sch (KiCad schematic)
At the start: 20 parts, among them J16 1x2 Goldpin Header, J17 1x2 Goldpin Header, J18 1x3 Goldpin Header, Q1 MMFTP3334K, U2 MCP1703A-3302E/DB

Commit message: optymalizacja BOM + pdf schematu
Parts:
- R3: renamed from R4; value 220R -> 240R; footprint Resistor_SMD:R_0603_1608Metric_Pad0.98x0.95mm_HandSolder -> Resistor_SMD:R_0805_2012Metric_Pad1.20x1.40mm_HandSolder; Package 0603 -> 0805; Part Number 0603SAJ0221T5E -> 0805S8J0241T5E
- renumbered R5 to R4
Changed lines of the file:
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@@
   (symbol (lib_id "Device:R") (at 53.34 105.41 0) (unit 1)
     (in_bom yes) (on_board yes) (dnp no)
-    (property "Reference" "R5" (at 55.88 104.14 0)
+    (property "Reference" "R4" (at 55.88 104.14 0)
       (effects (font (size 1.27 1.27)) (justify left))
     )
@@
       (project "ATXMEGA256_Miniboard"
         (path "/ef1e5883-c6cf-4bad-8eaa-8ec9109f9d71/1d37de11-1936-4242-b544-634b362ae3ca"
-          (reference "R5") (unit 1)
+          (reference "R4") (unit 1)
         )
       )
@@
   (symbol (lib_id "Device:R") (at 120.65 97.79 0) (unit 1)
     (in_bom yes) (on_board yes) (dnp no)
-    (property "Reference" "R4" (at 123.19 96.52 0)
-      (effects (font (size 1.27 1.27)) (justify left))
-    )
-    (property "Value" "220R" (at 123.19 99.06 0)
-      (effects (font (size 1.27 1.27)) (justify left))
-    )
-    (property "Footprint" "Resistor_SMD:R_0603_1608Metric_Pad0.98x0.95mm_HandSolder" (at 118.872 97.79 90)
+    (property "Reference" "R3" (at 123.19 96.52 0)
+      (effects (font (size 1.27 1.27)) (justify left))
+    )
+    (property "Value" "240R" (at 123.19 99.06 0)
+      (effects (font (size 1.27 1.27)) (justify left))
+    )
+    (property "Footprint" "Resistor_SMD:R_0805_2012Metric_Pad1.20x1.40mm_HandSolder" (at 118.872 97.79 90)
       (effects (font (size 1.27 1.27)) hide)
     )
@@
       (effects (font (size 1.27 1.27)) hide)
     )
-    (property "Part Number" "0603SAJ0221T5E" (at 120.65 97.79 0)
+    (property "Part Number" "0805S8J0241T5E" (at 120.65 97.79 0)
       (effects (font (size 1.27 1.27)) hide)
     )
@@
       (effects (font (size 1.27 1.27)) hide)
     )
-    (property "Package" "0603" (at 125.73 101.6 0)
-      (effects (font (size 1.27 1.27)) hide)
-    )
-    (pin "2")
-    (pin "1")
-    (instances
-      (project "ATXMEGA256_Miniboard"
-        (path "/ef1e5883-c6cf-4bad-8eaa-8ec9109f9d71/1d37de11-1936-4242-b544-634b362ae3ca"
-          (reference "R4") (unit 1)
-        )
-      )
+    (property "Package" "0805" (at 125.73 101.6 0)
+      (effects (font (size 1.27 1.27)) hide)
+    )
+    (pin "2")
+    (pin "1")
+    (instances
+      (project "ATXMEGA256_Miniboard"
+        (path "/ef1e5883-c6cf-4bad-8eaa-8ec9109f9d71/1d37de11-1936-4242-b544-634b362ae3ca"
+          (reference "R3") (unit 1)
+        )
+      )

Commit message: rev 1.1
Parts:
- removed C10, C11, C13, C7, C8, C9: 100n, Capacitor_SMD:C_0805_2012Metric_Pad1.18x1.45mm_HandSolder, symbol Device:C
- removed C12: 10u, Capacitor_SMD:C_1210_3225Metric_Pad1.33x2.70mm_HandSolder, symbol Device:C
- removed L2: 2u2, Inductor_SMD:L_0805_2012Metric_Pad1.15x1.40mm_HandSolder, symbol Device:L_Ferrite
- renumbered C4 to C12, C5 to C13, C6 to C14, J16 to J6, J17 to J7, J18 to J8, L1 to L2
Connections:
- net +3V3: now also C13.2, J6.2 (Pin_2), R3.1, U2.3 (VOUT); no longer J6.1 (Pin_1), L2.1
- net +3V3_MCU_VCC renamed VCC_MCU
- net EXT_VCC renamed VCC_EXT
- new net: J6.1 (Pin_1), L2.1
Other:
- note removed: "Kondensatory odsprzęgające pinów zasilających MCU"
- note removed: "Zasilanie części analogowej MCU"
- moved on the sheet: C12, C13, C14, D1, J6, J7, J8, L2, Q1, R3, R4, U2
