File: kicad/ATXMEGA256_Miniboard/ATXMEGA256_Miniboard.kicad_pcb (KiCad board)
At the start: 2 copper layers, 25 parts, among them J1 DS1021-2*3SF11-B, J2 ZL264-10DG, J3 ZL264-10DG, J4 ZL264-10DG, J5 ZL264-6DG, J6 ZL264-10DG, J7 ZL264-10DG, J8 ZL264-6DG, J9 JTAG, U1 ATXMEGA256A3B-AU

Commit message: v1.0
Parts:
- removed C1, C2, C3, C4, C5, C6: 100n, Capacitor_SMD:C_0805_2012Metric_Pad1.18x1.45mm_HandSolder
- removed C7, C8: 10p, Capacitor_SMD:C_0603_1608Metric_Pad1.08x0.95mm_HandSolder
- removed J1: DS1021-2*3SF11-B, Connector_PinHeader_2.54mm:PinHeader_2x03_P2.54mm_Vertical_SMD
- removed J2, J3, J4, J6, J7: ZL264-10DG, Connector_PinSocket_2.54mm:PinSocket_2x05_P2.54mm_Vertical_SMD
- removed J5, J8: ZL264-6DG, Connector_PinSocket_2.54mm:PinSocket_2x03_P2.54mm_Vertical_SMD
- removed J9: JTAG, Connector_IDC:IDC-Header_2x05_P2.54mm_Vertical
- removed JP1, JP3: DS1021-1X2SF162-B, Connector_PinHeader_2.54mm:PinHeader_1x02_P2.54mm_Vertical
- removed JP2, JP4: Solder Jumper, Jumper:SolderJumper-3_P1.3mm_Bridged12_Pad1.0x1.5mm_NumberLabels
- removed L1: 2u, Inductor_SMD:L_0805_2012Metric_Pad1.15x1.40mm_HandSolder
- removed R1: 10k, Resistor_SMD:R_0805_2012Metric_Pad1.20x1.40mm_HandSolder
- removed R2: 330R, Resistor_SMD:R_0805_2012Metric_Pad1.20x1.40mm_HandSolder
- removed U1: ATXMEGA256A3B-AU, ATXMega256A3B-AU:QFP80P1600X1600X120-64N

Commit message: usb + udokumentowanie elementów
Parts:
- added C1: 100n, Capacitor_SMD:C_0805_2012Metric_Pad1.18x1.45mm_HandSolder, F.Cu at (142.0, 75.9)
- added C2: 100n, Capacitor_SMD:C_0805_2012Metric_Pad1.18x1.45mm_HandSolder, F.Cu at (142.0, 78.9)
- added C3: 100n, Capacitor_SMD:C_0805_2012Metric_Pad1.18x1.45mm_HandSolder, F.Cu at (142.0, 81.9)
- added C4: 100n, Capacitor_SMD:C_0805_2012Metric_Pad1.18x1.45mm_HandSolder, F.Cu at (142.0, 84.9)
- added C5: 100n, Capacitor_SMD:C_0805_2012Metric_Pad1.18x1.45mm_HandSolder, F.Cu at (142.0, 87.9)
- added C6: 10u, Capacitor_SMD:C_1210_3225Metric_Pad1.33x2.70mm_HandSolder, F.Cu at (152.1, 94.1)
- added C7: 100n, Capacitor_SMD:C_0805_2012Metric_Pad1.18x1.45mm_HandSolder, F.Cu at (142.0, 90.9)
- added C8: 12p, Capacitor_SMD:C_0603_1608Metric_Pad1.08x0.95mm_HandSolder, F.Cu at (146.6, 90.4)
- added C9: 12p, Capacitor_SMD:C_0603_1608Metric_Pad1.08x0.95mm_HandSolder, F.Cu at (146.6, 92.9)
- added J1: DS1013-10SSIB1-B-0, Connector_IDC:IDC-Header_2x05_P2.54mm_Vertical, F.Cu at (122.7, 73.3)
- added J10: USB_B_Micro, Connector_USB:USB_Micro-AB_Molex_47590-0001, F.Cu at (154.8, 88.8)
- added J2: DS1021-2*3SF11-B, Connector_PinHeader_2.54mm:PinHeader_2x03_P2.54mm_Vertical_SMD, F.Cu at (155.6, 79.2)
- added J3: ZL264-10DG, Connector_PinSocket_2.54mm:PinSocket_2x05_P2.54mm_Vertical_SMD, F.Cu at (122.6, 59.8)
- added J4: ZL264-10DG, Connector_PinSocket_2.54mm:PinSocket_2x05_P2.54mm_Vertical_SMD, F.Cu at (132.7, 59.8)
- added J5: ZL264-10DG, Connector_PinSocket_2.54mm:PinSocket_2x05_P2.54mm_Vertical_SMD, F.Cu at (142.8, 59.8)
- added J6: ZL264-6DG, Connector_PinSocket_2.54mm:PinSocket_2x03_P2.54mm_Vertical_SMD, F.Cu at (134.5, 72.0)
- added J7: ZL264-10DG, Connector_PinSocket_2.54mm:PinSocket_2x05_P2.54mm_Vertical_SMD, F.Cu at (152.9, 59.8)
- added J8: ZL264-10DG, Connector_PinSocket_2.54mm:PinSocket_2x05_P2.54mm_Vertical_SMD, F.Cu at (163.0, 59.8)
- added J9: ZL264-6DG, Connector_PinSocket_2.54mm:PinSocket_2x03_P2.54mm_Vertical_SMD, F.Cu at (134.5, 81.7)
- added JP1: DS1021-1X2SF162-B, Connector_PinHeader_2.54mm:PinHeader_1x02_P2.54mm_Vertical, F.Cu at (141.9, 69.5)
- added JP2: Solder Jumper, Jumper:SolderJumper-3_P1.3mm_Bridged12_Pad1.0x1.5mm_NumberLabels, F.Cu at (164.8, 76.1)
- added JP3: DS1021-1X2SF162-B, Connector_PinHeader_2.54mm:PinHeader_1x02_P2.54mm_Vertical, F.Cu at (146.5, 69.5)
- added JP4: Solder Jumper, Jumper:SolderJumper-3_P1.3mm_Bridged12_Pad1.0x1.5mm_NumberLabels, F.Cu at (164.8, 79.7)
- added JP5: DS1021-1X2SF162-B, Connector_PinHeader_2.54mm:PinHeader_1x02_P2.54mm_Vertical, F.Cu at (151.2, 69.5)
- added JP6: DS1021-1X2SF162-B, Connector_PinHeader_2.54mm:PinHeader_1x02_P2.54mm_Vertical, F.Cu at (155.8, 69.5)
- added L1: 2u, Inductor_SMD:L_0805_2012Metric_Pad1.15x1.40mm_HandSolder, F.Cu at (146.8, 75.8)
- added R1: 10k, Resistor_SMD:R_0805_2012Metric_Pad1.20x1.40mm_HandSolder, F.Cu at (146.8, 78.8)
- added R2: 330R, Resistor_SMD:R_0805_2012Metric_Pad1.20x1.40mm_HandSolder, F.Cu at (146.8, 81.7)
- added R3: 22R, Resistor_SMD:R_0805_2012Metric_Pad1.20x1.40mm_HandSolder, F.Cu at (146.8, 84.7)
- added R4: 22R, Resistor_SMD:R_0805_2012Metric_Pad1.20x1.40mm_HandSolder, F.Cu at (146.8, 87.6)
- added SW1: 1301.9303, Button_Switch_THT:SW_PUSH_6mm_H7.3mm, F.Cu at (119.5, 91.6)
- added U1: ATXMEGA256A3B-AU, ATXMega256A3B-AU:QFP80P1600X1600X120-64N, F.Cu at (136.4, 109.3)
- added Y1: LFXTAL014219, Crystal:Crystal_DS26_D2.0mm_L6.0mm_Horizontal_1EP_style1, F.Cu at (161.9, 85.4)
- added Y2: LFXTAL053426, Crystal:Crystal_SMD_3225-4Pin_3.2x2.5mm, F.Cu at (157.8, 94.2)
Other:
- board outline added: 7.5 x 2 mm

Commit message: przycisk zmieniony na smd
Parts:
- removed C1, C2, C3, C4, C5, C7: 100n, Capacitor_SMD:C_0805_2012Metric_Pad1.18x1.45mm_HandSolder
- removed C6: 10u, Capacitor_SMD:C_1210_3225Metric_Pad1.33x2.70mm_HandSolder
- removed C8, C9: 12p, Capacitor_SMD:C_0603_1608Metric_Pad1.08x0.95mm_HandSolder
- removed J1: DS1013-10SSIB1-B-0, Connector_IDC:IDC-Header_2x05_P2.54mm_Vertical
- removed J10: USB_B_Micro, Connector_USB:USB_Micro-AB_Molex_47590-0001
- removed J2: DS1021-2*3SF11-B, Connector_PinHeader_2.54mm:PinHeader_2x03_P2.54mm_Vertical_SMD
- removed J3, J4, J5, J7, J8: ZL264-10DG, Connector_PinSocket_2.54mm:PinSocket_2x05_P2.54mm_Vertical_SMD
- removed J6, J9: ZL264-6DG, Connector_PinSocket_2.54mm:PinSocket_2x03_P2.54mm_Vertical_SMD
- removed JP1, JP3, JP5, JP6: DS1021-1X2SF162-B, Connector_PinHeader_2.54mm:PinHeader_1x02_P2.54mm_Vertical
- removed JP2, JP4: Solder Jumper, Jumper:SolderJumper-3_P1.3mm_Bridged12_Pad1.0x1.5mm_NumberLabels
- removed L1: 2u, Inductor_SMD:L_0805_2012Metric_Pad1.15x1.40mm_HandSolder
- removed R1: 10k, Resistor_SMD:R_0805_2012Metric_Pad1.20x1.40mm_HandSolder
- removed R2: 330R, Resistor_SMD:R_0805_2012Metric_Pad1.20x1.40mm_HandSolder
- removed R3, R4: 22R, Resistor_SMD:R_0805_2012Metric_Pad1.20x1.40mm_HandSolder
- removed SW1: 1301.9303, Button_Switch_THT:SW_PUSH_6mm_H7.3mm
- removed U1: ATXMEGA256A3B-AU, ATXMega256A3B-AU:QFP80P1600X1600X120-64N
- removed Y1: LFXTAL014219, Crystal:Crystal_DS26_D2.0mm_L6.0mm_Horizontal_1EP_style1
- removed Y2: LFXTAL053426, Crystal:Crystal_SMD_3225-4Pin_3.2x2.5mm
Other:
- board outline removed

Commit message: pdated parts on PCB from schematic, migrated to kicad 9
Parts:
- added C1: 100n, Capacitor_SMD:C_0805_2012Metric_Pad1.18x1.45mm_HandSolder, F.Cu at (57.8, 149.5)
- added C10: 12p, Capacitor_SMD:C_0603_1608Metric_Pad1.08x0.95mm_HandSolder, F.Cu at (75.6, 161.5)
- added C11: 12p, Capacitor_SMD:C_0603_1608Metric_Pad1.08x0.95mm_HandSolder, F.Cu at (75.6, 164.0)
- added C12: 10u, Capacitor_SMD:C_1210_3225Metric_Pad1.33x2.70mm_HandSolder, F.Cu at (95.8, 129.6)
- added C13: 10u, Capacitor_SMD:C_1210_3225Metric_Pad1.33x2.70mm_HandSolder, F.Cu at (95.8, 133.9)
- added C14: 10u, Capacitor_SMD:C_1210_3225Metric_Pad1.33x2.70mm_HandSolder, F.Cu at (95.8, 138.1)
- added C2: 100n, Capacitor_SMD:C_0805_2012Metric_Pad1.18x1.45mm_HandSolder, F.Cu at (57.8, 152.6)
- added C3: 100n, Capacitor_SMD:C_0805_2012Metric_Pad1.18x1.45mm_HandSolder, F.Cu at (57.8, 155.6)
- added C4: 100n, Capacitor_SMD:C_0805_2012Metric_Pad1.18x1.45mm_HandSolder, F.Cu at (57.8, 158.6)
- added C5: 100n, Capacitor_SMD:C_0805_2012Metric_Pad1.18x1.45mm_HandSolder, F.Cu at (57.8, 161.6)
- added C6: 10u, Capacitor_SMD:C_1210_3225Metric_Pad1.33x2.70mm_HandSolder, F.Cu at (76.0, 150.2)
- added C7: 100n, Capacitor_SMD:C_0805_2012Metric_Pad1.18x1.45mm_HandSolder, F.Cu at (57.8, 164.6)
- added C8: 100n, Capacitor_SMD:C_0805_2012Metric_Pad1.18x1.45mm_HandSolder, F.Cu at (57.8, 167.6)
- added C9: 4n7, Capacitor_SMD:C_0603_1608Metric_Pad1.08x0.95mm_HandSolder, F.Cu at (75.6, 159.0)
- added D1: RED LED, LED_SMD:LED_0805_2012Metric_Pad1.15x1.40mm_HandSolder, F.Cu at (100.2, 141.8)
- added J1: 1x2 Screw Terminal, TerminalBlock:TerminalBlock_bornier-2_P5.08mm, F.Cu at (67.2, 132.0)
- added J10: 2x5 Goldpin Socket, Connector_PinSocket_2.54mm:PinSocket_2x05_P2.54mm_Vertical_SMD, F.Cu at (58.6, 108.4)
- added J11: 2x5 Goldpin Socket, Connector_PinSocket_2.54mm:PinSocket_2x05_P2.54mm_Vertical_SMD, F.Cu at (68.7, 108.4)
- added J12: 2x3 Goldpin Socket, Connector_PinSocket_2.54mm:PinSocket_2x03_P2.54mm_Vertical_SMD, F.Cu at (48.5, 120.7)
- added J13: 2x5 Goldpin Socket, Connector_PinSocket_2.54mm:PinSocket_2x05_P2.54mm_Vertical_SMD, F.Cu at (78.8, 108.4)
- added J14: 2x5 Goldpin Socket, Connector_PinSocket_2.54mm:PinSocket_2x05_P2.54mm_Vertical_SMD, F.Cu at (88.9, 108.4)
- added J2: 10118192-0001LF, 10118192-0001LF:AMPHENOL_10118192-0001LF, F.Cu at (65.7, 159.8)
- added J3: 2x5 IDC Socket, Connector_IDC:IDC-Header_2x05_P2.54mm_Vertical, F.Cu at (48.7, 154.2)
- added J4: 2x3 Goldpin Socket, Connector_PinSocket_2.54mm:PinSocket_2x03_P2.54mm_Vertical_SMD, F.Cu at (69.0, 141.4)
- added J5: 2x3 Goldpin Header, Connector_PinHeader_2.54mm:PinHeader_2x03_P2.54mm_Vertical_SMD, F.Cu at (66.6, 152.9)
- added J6: 1x2 Goldpin Header, Connector_PinHeader_2.54mm:PinHeader_1x02_P2.54mm_Vertical, F.Cu at (85.4, 138.7)
- added J7: 1x2 Goldpin Header, Connector_PinHeader_2.54mm:PinHeader_1x02_P2.54mm_Vertical, F.Cu at (90.0, 138.7)
- added J8: 1x3 Goldpin Header, Connector_PinHeader_2.54mm:PinHeader_1x03_P2.54mm_Vertical, F.Cu at (101.1, 129.8)
- added J9: 2x5 Goldpin Socket, Connector_PinSocket_2.54mm:PinSocket_2x05_P2.54mm_Vertical_SMD, F.Cu at (48.5, 108.4)
- added JP1: Solder Jumper, Jumper:SolderJumper-3_P1.3mm_Bridged12_RoundedPad1.0x1.5mm_NumberLabels, F.Cu at (78.3, 129.3)
- added JP2: Solder Jumper, Jumper:SolderJumper-3_P1.3mm_Bridged12_RoundedPad1.0x1.5mm_NumberLabels, F.Cu at (78.3, 132.8)
- added L1: 2u2, Inductor_SMD:L_0805_2012Metric_Pad1.15x1.40mm_HandSolder, F.Cu at (57.8, 170.6)
- added L2: 10u, Inductor_SMD:L_0805_2012Metric_Pad1.05x1.20mm_HandSolder, F.Cu at (100.2, 144.7)
- added Q1: MMFTP3334K, MMFTP3334K:TRANS_MMFTP3334K, F.Cu at (95.5, 142.5)
- added R1: 10k, Resistor_SMD:R_0603_1608Metric_Pad0.98x0.95mm_HandSolder, F.Cu at (75.6, 166.5)
- added R2: 1M, Resistor_SMD:R_0603_1608Metric_Pad0.98x0.95mm_HandSolder, F.Cu at (75.6, 169.0)
- added R3: 240R, Resistor_SMD:R_0805_2012Metric_Pad1.20x1.40mm_HandSolder, F.Cu at (101.2, 138.6)
- added R4: 10k, Resistor_SMD:R_0603_1608Metric_Pad0.98x0.95mm_HandSolder, F.Cu at (85.3, 144.8)
- added SW1: RESET, Button_Switch_SMD:SW_SPST_Omron_B3FS-100xP, F.Cu at (65.9, 169.9)
- added U1: ATXMEGA256A3B-AU, ATXMega256A3B-AU:QFP80P1600X1600X120-64N, F.Cu at (53.7, 137.8)
- added U2: MCP1703A-3302E/DB, MCP1703A-3302E:SOT230P700X180-4N, F.Cu at (88.0, 132.2)
- added Y1: 32.768 kHz, Crystal:Crystal_DS26_D2.0mm_L6.0mm_Horizontal_1EP_style1, F.Cu at (75.4, 137.8)
- added Y2: 16 MHz, Crystal:Crystal_SMD_3225-4Pin_3.2x2.5mm, F.Cu at (75.7, 154.6)
