File: kicad/ATXMEGA256_Miniboard/ATXMEGA256_Miniboard_v2.kicad_pcb (KiCad board)
At the start: 4 copper layers, 50 x 70 mm, 42 parts, among them J1 1x2 Screw Terminal, J10 2x5 Goldpin Socket, J11 2x5 Goldpin Socket, J12 2x3 Goldpin Socket, J13 2x5 Goldpin Socket, J14 2x5 Goldpin Socket, J2 10118192-0001LF, J3 2x5 IDC Socket, J4 2x3 Goldpin Socket, J5 2x3 Goldpin Header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

Commit message: PCB layout
Parts:
- moved J4 64.9 mm to (59.5, 132.2), turned to 90 degrees
- moved J3 63.7 mm to (36.8, 192.8), turned to 90 degrees
- moved Y1 36.3 mm to (55.5, 154.4), turned to 90 degrees
- moved J5 9.57 mm to (59.5, 143.5), turned to 90 degrees
- moved J14 0.45 mm to (59.7, 188.7)
- moved J13 0.41 mm to (59.8, 174.2)
- moved J12 0.38 mm to (59.8, 162.2)
Routing:
- net /PB6: track 78.2 -> 32.0 mm, vias 1 -> 2
- net /PB7: track 81.1 -> 35.7 mm, vias 2 -> 4
- net /~{RESET}: track 58.6 -> 96.2 mm, vias 0 -> 4
- net /PB4: track 69.8 -> 36.4 mm, vias 1 -> 2
- net /PB5: track 69.8 -> 46.0 mm, vias 2 -> 3
- net /PF0: track 30.9 -> 49.5 mm
- net /PF1: track 25.4 -> 43.6 mm
- net /PF2: track 34.6 -> 52.4 mm, vias 0 -> 2
- net /PF6: track 48.7 -> 64.3 mm
- net /VBAT: track 40.1 -> 54.2 mm
- net /PF7: track 42.3 -> 56.2 mm, vias 0 -> 2
- net +3V3: track 199.0 -> 186.0 mm, vias 9 -> 8
- net /PE0: track 26.0 -> 38.3 mm, vias 2 -> 0
- net /PF4: track 45.8 -> 57.9 mm
- net /PF3: track 38.0 -> 48.4 mm
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- added copper zone on In2.Cu, net +3V3
- added copper zone on In2.Cu, net +5V
- added copper zone on In2.Cu, net /Power Supply/VCC_EXT
- added copper zone on In2.Cu, net /Power Supply/VCC_MCU
- added copper zone on In2.Cu, net Net-(J8-Pin_2)
- added copper zone on In2.Cu, net Net-(U1-AVCC)
